File: output/pcbs/left_pcb.kicad_pcb (KiCad board)
At the start: 2 copper layers, 132 x 117.7 mm, 37 parts

Commit message: fix spacing
Parts:
- moved D15 20.4 mm to (172.0, 68.5)
- moved S15 20.4 mm to (172.0, 63.5)
- moved D12 20.2 mm to (154.0, 66.0)
- moved S12 20.2 mm to (154.0, 61.0)
- moved D9 20.1 mm to (136.0, 63.5)
- moved S9 20.1 mm to (136.0, 58.5)
- moved D6 20.0 mm to (118.0, 66.0)
- moved S6 20.0 mm to (118.0, 61.0)
- moved D3 20.0 mm to (100.0, 71.0)
- moved S3 20.0 mm to (100.0, 66.0)
- moved B1 10.8 mm to (207.0, 95.5)
- moved D14 10.8 mm to (172.0, 85.5)
- moved MCU1 10.8 mm to (202.0, 72.5)
- moved S14 10.8 mm to (172.0, 80.5)
- moved D11 10.4 mm to (154.0, 83.0)
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Routing:
- net GND: track 61.0 -> 22.8 mm
- net L_R2: track 214.9 -> 178.8 mm
- net L_C1: track 178.4 -> 143.5 mm
- net L_C2: track 158.2 -> 126.1 mm
- net L_R3: track 121.7 -> 95.5 mm
- net L_C3: track 137.1 -> 111.2 mm
- net L_C0: track 183.9 -> 163.8 mm
- net L_T1: track 81.5 -> 63.9 mm
- net L_R1: track 195.6 -> 184.1 mm
- net L_C4: track 116.0 -> 105.2 mm
- net L_T0: track 87.8 -> 77.4 mm
- net L_R0: track 199.2 -> 192.5 mm
- net SERIAL: track 34.8 -> 31.0 mm
- net VCC: track 76.4 -> 74.1 mm
- net RST: track 42.2 -> 41.2 mm
Other:
- board size 132 x 117.7 mm -> 128 x 97.5 mm

Commit message: Refactor keyboard.yaml to remove reset button configurations, update PCB net patterns for left and right PCBs, and adjust matrix pin assignments in info.json. Enhance README with stagger details for both hands.
Parts:
- removed B1: , E73:SW_TACT_ALPS_SKQGABE010
- moved TRRS1 4.80 mm to (207.0, 102.5)
Connections:
- D1 pad 1: L_C0 -> left_matrix_pinky_bottom
- D10 pad 1: L_C3 -> left_matrix_index_bottom
- D11 pad 1: L_C3 -> left_matrix_index_home
- D12 pad 1: L_C3 -> left_matrix_index_top
- D13 pad 1: L_C4 -> left_matrix_inner_bottom
- D14 pad 1: L_C4 -> left_matrix_inner_home
- D15 pad 1: L_C4 -> left_matrix_inner_top
- D16 pad 1: L_T0 -> left_thumb_outer_thumb
- D17 pad 1: L_T1 -> left_thumb_inner_thumb
- D2 pad 1: L_C0 -> left_matrix_pinky_home
- D3 pad 1: L_C0 -> left_matrix_pinky_top
- D4 pad 1: L_C1 -> left_matrix_ring_bottom
- D5 pad 1: L_C1 -> left_matrix_ring_home
- D6 pad 1: L_C1 -> left_matrix_ring_top
- D7 pad 1: L_C2 -> left_matrix_middle_bottom
- D8 pad 1: L_C2 -> left_matrix_middle_home
- D9 pad 1: L_C2 -> left_matrix_middle_top
- S1 pad 2: L_R0 -> left_matrix_pinky_bottom
- S10 pad 2: L_R0 -> left_matrix_index_bottom
- S11 pad 2: L_R1 -> left_matrix_index_home
- S12 pad 2: L_R2 -> left_matrix_index_top
- S13 pad 2: L_R0 -> left_matrix_inner_bottom
- S14 pad 2: L_R1 -> left_matrix_inner_home
- S15 pad 2: L_R2 -> left_matrix_inner_top
- S16 pad 2: L_R3 -> left_thumb_outer_thumb
- S17 pad 2: L_R3 -> left_thumb_inner_thumb
- S2 pad 2: L_R1 -> left_matrix_pinky_home
- S3 pad 2: L_R2 -> left_matrix_pinky_top
- S4 pad 2: L_R0 -> left_matrix_ring_bottom
- S5 pad 2: L_R1 -> left_matrix_ring_home
- S6 pad 2: L_R2 -> left_matrix_ring_top
- S7 pad 2: L_R0 -> left_matrix_middle_bottom
- S8 pad 2: L_R1 -> left_matrix_middle_home
- S9 pad 2: L_R2 -> left_matrix_middle_top
Routing:
- net L_R0: track 192.5 -> 0.00 mm
- net L_R1: track 184.1 -> 0.00 mm
- net L_R2: track 178.8 -> 0.00 mm
- net L_C0: track 163.8 -> 0.00 mm
- net L_C1: track 143.5 -> 0.00 mm
- net L_C2: track 126.1 -> 0.00 mm
- net L_C3: track 111.2 -> 0.00 mm
- net L_C4: track 105.2 -> 0.00 mm
- net L_R3: track 95.5 -> 0.00 mm
- net L_T0: track 77.4 -> 0.00 mm
- net VCC: track 74.1 -> 0.00 mm
- net L_T1: track 63.9 -> 0.00 mm
- net RST: track 41.2 -> 0.00 mm
- net SERIAL: track 31.0 -> 0.00 mm
- net GND: track 22.8 -> 0.00 mm
- removed copper zone on B.Cu, net GND
Other:
- net class Default added: clearance 0.2, trace_width 0.25, via_dia 0.8, via_drill 0.4
