File: output/pcbs/right_pcb.kicad_pcb (KiCad board)
At the start: 2 copper layers, 132 x 113 mm, 35 parts

Commit message: fix spacing
Parts:
- moved D12 20.2 mm to (154.0, 73.5)
- moved S12 20.2 mm to (154.0, 68.5)
- moved D9 20.1 mm to (136.0, 68.5)
- moved S9 20.1 mm to (136.0, 63.5)
- moved D6 20.0 mm to (118.0, 66.0)
- moved S6 20.0 mm to (118.0, 61.0)
- moved D3 20.0 mm to (100.0, 68.5)
- moved S3 20.0 mm to (100.0, 63.5)
- moved D14 10.8 mm to (172.0, 90.5)
- moved S14 10.8 mm to (172.0, 85.5)
- moved D11 10.4 mm to (154.0, 90.5)
- moved S11 10.4 mm to (154.0, 85.5)
- moved D8 10.2 mm to (136.0, 85.5)
- moved S8 10.2 mm to (136.0, 80.5)
- moved D5 10.0 mm to (118.0, 83.0)
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Routing:
- net R_R3: track 150.0 -> 105.4 mm
- net GND: track 57.3 -> 18.0 mm
- net R_C2: track 147.1 -> 121.8 mm
- net R_C0: track 101.8 -> 77.7 mm
- net R_C1: track 122.9 -> 100.9 mm
- net R_C3: track 159.9 -> 140.2 mm
- net R_C4: track 160.1 -> 143.8 mm
- net RST: track 57.1 -> 68.1 mm
- net R_R2: track 174.7 -> 164.6 mm
- net SERIAL: track 33.8 -> 23.8 mm
- net VCC: track 59.4 -> 49.8 mm
- net R_R1: track 209.9 -> 206.1 mm
- net R_R0: track 212.1 -> 209.9 mm
- net R_T1: track 62.9 -> 64.8 mm
- net R_T0: track 66.7 -> 67.7 mm
Other:
- board size 132 x 113 mm -> 128 x 92.7 mm
- board text removed: "安心"

Commit message: Refactor keyboard.yaml to remove reset button configurations, update PCB net patterns for left and right PCBs, and adjust matrix pin assignments in info.json. Enhance README with stagger details for both hands.
Parts:
- removed B1: , E73:SW_TACT_ALPS_SKQGABE010
Connections:
- D1 pad 1: R_C0 -> right_matrix_inner_bottom
- D10 pad 1: R_C3 -> right_matrix_ring_bottom
- D11 pad 1: R_C3 -> right_matrix_ring_home
- D12 pad 1: R_C3 -> right_matrix_ring_top
- D13 pad 1: R_C4 -> right_matrix_pinky_bottom
- D14 pad 1: R_C4 -> right_matrix_pinky_home
- D15 pad 1: R_T0 -> right_thumb_outer_thumb
- D16 pad 1: R_T1 -> right_thumb_inner_thumb
- D2 pad 1: R_C0 -> right_matrix_inner_home
- D3 pad 1: R_C0 -> right_matrix_inner_top
- D4 pad 1: R_C1 -> right_matrix_index_bottom
- D5 pad 1: R_C1 -> right_matrix_index_home
- D6 pad 1: R_C1 -> right_matrix_index_top
- D7 pad 1: R_C2 -> right_matrix_middle_bottom
- D8 pad 1: R_C2 -> right_matrix_middle_home
- D9 pad 1: R_C2 -> right_matrix_middle_top
- MCU1 pad 22: R_R2 -> R_R0
- MCU1 pad 24: R_R0 -> R_R2
- S1 pad 2: R_R0 -> right_matrix_inner_bottom
- S10 pad 2: R_R0 -> right_matrix_ring_bottom
- S11 pad 2: R_R1 -> right_matrix_ring_home
- S12 pad 2: R_R2 -> right_matrix_ring_top
- S13 pad 2: R_R0 -> right_matrix_pinky_bottom
- S14 pad 2: R_R1 -> right_matrix_pinky_home
- S15 pad 2: R_R3 -> right_thumb_outer_thumb
- S16 pad 2: R_R3 -> right_thumb_inner_thumb
- S2 pad 2: R_R1 -> right_matrix_inner_home
- S3 pad 2: R_R2 -> right_matrix_inner_top
- S4 pad 2: R_R0 -> right_matrix_index_bottom
- S5 pad 2: R_R1 -> right_matrix_index_home
- S6 pad 2: R_R2 -> right_matrix_index_top
- S7 pad 2: R_R0 -> right_matrix_middle_bottom
- S8 pad 2: R_R1 -> right_matrix_middle_home
- S9 pad 2: R_R2 -> right_matrix_middle_top
Routing:
- net R_R0: track 209.9 -> 0.00 mm
- net R_R1: track 206.1 -> 0.00 mm
- net R_R2: track 164.6 -> 0.00 mm
- net R_C4: track 143.8 -> 0.00 mm
- net R_C3: track 140.2 -> 0.00 mm
- net R_C2: track 121.8 -> 0.00 mm
- net R_R3: track 105.4 -> 0.00 mm
- net R_C1: track 100.9 -> 0.00 mm
- net R_C0: track 77.7 -> 0.00 mm
- net RST: track 68.1 -> 0.00 mm
- net R_T0: track 67.7 -> 0.00 mm
- net R_T1: track 64.8 -> 0.00 mm
- net VCC: track 49.8 -> 0.00 mm
- net SERIAL: track 23.8 -> 0.00 mm
- net GND: track 18.0 -> 0.00 mm
- removed copper zone on B.Cu, net GND
Other:
- net class Default added: clearance 0.2, trace_width 0.25, via_dia 0.8, via_drill 0.4
